File: OpenAmigaMouseTrigger.sch (KiCad schematic (older format))
At the start: 8 parts, among them J1 AMIGA_SIGNALS, J2 OUTPUT, J3 POWER, J99 OSHW_LOGO, U1 74LS74

Commit message: Final touches for V1
Parts:
- added R2, R3: 22k, Resistors_THT:R_Axial_DIN0207_L6.3mm_D2.5mm_P10.16mm_Horizontal, symbol R
- R1: value 10k -> 4.7k
Connections:
- net VCC: now also R2.1, R3.1
- net at J1.1 (Pin_1), U1.2 (D): now also R2.2
- net at J1.2 (Pin_2), U1.12 (D): now also R3.2
Other:
- note added: "OPTIONAL Weak\nPull-Up Resistors"
- moved on the sheet: J1
Changed lines of the file:
@@
 LIBS:contrib
 LIBS:valves
+LIBS:OpenAmigaMouseTrigger-cache
 EELAYER 25 0
 EELAYER END
@@
 Sheet 1 1
 Title "OpenAmigaMouseTrigger"
-Date "2017-12-18"
-Rev "20171218"
+Date "2018-01-07"
+Rev "1"
 Comp "SukkoPera"
 Comment1 ""
@@
 L Conn_01x02 J1
 U 1 1 5A383421
-P 4175 3925
-F 0 "J1" H 4175 4025 50  0000 C CNN
-F 1 "AMIGA_SIGNALS" H 4225 3725 50  0000 C CNN
-F 2 "OpenAmigaMouseTrigger:LoosePads-2" H 4175 3925 50  0001 C CNN
-F 3 "" H 4175 3925 50  0001 C CNN
-	1    4175 3925
+P 3750 3925
+F 0 "J1" H 3750 4025 50  0000 C CNN
+F 1 "AMIGA_SIGNALS" H 3800 3725 50  0000 C CNN
+F 2 "OpenAmigaMouseTrigger:LoosePads-2" H 3750 3925 50  0001 C CNN
+F 3 "" H 3750 3925 50  0001 C CNN
+	1    3750 3925
 	-1   0    0    -1
 $EndComp
-Text Notes 3300 3950 0    50   ~ 0
+Text Notes 2875 3950 0    50   ~ 0
 LMB (Odd CIA Pin 8)
-Text Notes 3325 4050 0    50   ~ 0
+Text Notes 2900 4050 0    50   ~ 0
 RMB (Paula Pin 33)
 $Comp
@@
 P 3850 4525
 F 0 "R1" V 3930 4525 50  0000 C CNN
-F 1 "10k" V 3850 4525 50  0000 C CNN
+F 1 "4.7k" V 3850 4525 50  0000 C CNN
 F 2 "Resistors_THT:R_Axial_DIN0207_L6.3mm_D2.5mm_P10.16mm_Horizontal" V 3780 4525 50  0001 C CNN
 F 3 "" H 3850 4525 50  0001 C CNN
@@
 	1    0    0    -1
 $EndComp
-Wire Wire Line
-	3475 4400 3475 4525
-Wire Wire Line
-	3475 4525 3700 4525
-Wire Wire Line
-	4000 4525 4875 4525
-Wire Wire Line
-	4875 3425 4875 4800
-Wire Wire Line
-	4875 4800 5400 4800
-Wire Wire Line
-	4875 3425 5400 3425
-Connection ~ 4875 4525
 $Comp
 L VCC #PWR02
@@
 	1    0    0    -1
 $EndComp
-Wire Wire Line
-	5200 2700 5200 5525
-Wire Wire Line
-	5200 2700 6000 2700
-Wire Wire Line
-	6000 2525 6000 2875
-Connection ~ 6000 2700
-Wire Wire Line
-	5200 4100 6000 4100
-Wire Wire Line
-	6000 3975 6000 4250
-Connection ~ 6000 4100
-Wire Wire Line
-	4375 3925 4750 3925
-Wire Wire Line
-	4750 3925 4750 3225
-Wire Wire Line
-	4750 4025 4750 4600
-Wire Wire Line
-	4750 3225 5400 3225
-Wire Wire Line
-	4750 4600 5400 4600
-Wire Wire Line
-	5200 5525 6000 5525
-Wire Wire Line
-	6000 5525 6000 5350
-Connection ~ 5200 4100
-Wire Wire Line
-	4375 4025 4750 4025
 NoConn ~ 6600 3625
 NoConn ~ 6600 5000
@@
 	1    0    0    -1
 $EndComp
-Wire Wire Line
-	6600 3225 7025 3225
-Wire Wire Line
-	7025 3225 7025 3925
-Wire Wire Line
-	7025 3925 7300 3925
-Wire Wire Line
-	7300 4025 7000 4025
-Wire Wire Line
-	7000 4025 7000 4600
-Wire Wire Line
-	7000 4600 6600 4600
 $Comp
 L C C2
@@
 	1    0    0    -1
 $EndComp
-Wire Wire Line
-	9400 3700 9400 3800
-Wire Wire Line
-	9400 4100 9400 4200
 $Comp
 L GND #PWR05
@@
 	-1   0    0    1
 $EndComp
-Wire Wire Line
-	10475 925  10475 825
-Wire Wire Line
-	10800 825  10800 900
 $Comp
 L Conn_01x02 J3
@@
 	1    0    0    -1
 $EndComp
-Wire Wire Line
-	10350 4100 10350 3950
 $Comp
 L GND #PWR010
@@
 	1    0    0    -1
 $EndComp
-Wire Wire Line
-	10450 4100 10450 4000
-Wire Wire Line
-	10450 4000 10775 4000
-Wire Wire Line
-	10775 4000 10775 4100
 Text Notes 3500 4825 0    60   ~ 0
 CLOCK PULSE\nGENERATOR
-Connection ~ 4275 4525
 $Comp
 L GND #PWR011
@@
 	1    0    0    -1
 $EndComp
-Wire Wire Line
-	4275 5075 4275 4975
-Wire Wire Line
-	4275 4525 4275 4675
 $Comp
 L Conn_01x01 J99
@@
 $EndComp
 NoConn ~ 10950 6075
+$Comp
+L R R2
+U 1 1 5A528FE1
+P 4150 3650
+F 0 "R2" V 4230 3650 50  0000 C CNN
+F 1 "22k" V 4150 3650 50  0000 C CNN
+F 2 "Resistors_THT:R_Axial_DIN0207_L6.3mm_D2.5mm_P10.16mm_Horizontal" V 4080 3650 50  0001 C CNN
+F 3 "" H 4150 3650 50  0001 C CNN
+	1    4150 3650
+	1    0    0    -1
+$EndComp
+$Comp
+L R R3
+U 1 1 5A5291EB
+P 4400 3650
+F 0 "R3" V 4480 3650 50  0000 C CNN
+F 1 "22k" V 4400 3650 50  0000 C CNN
+F 2 "Resistors_THT:R_Axial_DIN0207_L6.3mm_D2.5mm_P10.16mm_Horizontal" V 4330 3650 50  0001 C CNN
+F 3 "" H 4400 3650 50  0001 C CNN
+	1    4400 3650
+	1    0    0    -1
+$EndComp
+Wire Wire Line
+	3475 4400 3475 4525
+Wire Wire Line
+	3475 4525 3700 4525
+Wire Wire Line
+	4000 4525 4875 4525
+Wire Wire Line
+	4875 3425 4875 4800
+Wire Wire Line
+	4875 4800 5400 4800
+Wire Wire Line
+	4875 3425 5400 3425
+Connection ~ 4875 4525
+Wire Wire Line
+	5200 2700 5200 5525
+Wire Wire Line
+	4150 2700 6000 2700
+Wire Wire Line
+	6000 2525 6000 2875
+Connection ~ 6000 2700
+Wire Wire Line
+	5200 4100 6000 4100
+Wire Wire Line
+	6000 3975 6000 4250
+Connection ~ 6000 4100
+Wire Wire Line
+	3950 3925 4750 3925
+Wire Wire Line
+	4750 3925 4750 3225
+Wire Wire Line
+	4750 4025 4750 4600
+Wire Wire Line
+	4750 3225 5400 3225
+Wire Wire Line
+	4750 4600 5400 4600
+Wire Wire Line
+	5200 5525 6000 5525
+Wire Wire Line
+	6000 5525 6000 5350
+Connection ~ 5200 4100
+Wire Wire Line
+	3950 4025 4750 4025
+Wire Wire Line
+	6600 3225 7025 3225
+Wire Wire Line
+	7025 3225 7025 3925
+Wire Wire Line
+	7025 3925 7300 3925
+Wire Wire Line
+	7300 4025 7000 4025
+Wire Wire Line
+	7000 4025 7000 4600
+Wire Wire Line
+	7000 4600 6600 4600
+Wire Wire Line
+	9400 3700 9400 3800
+Wire Wire Line
+	9400 4100 9400 4200
+Wire Wire Line
+	10475 925  10475 825
+Wire Wire Line
+	10800 825  10800 900
+Wire Wire Line
+	10350 4100 10350 3950
+Wire Wire Line
+	10450 4100 10450 4000
+Wire Wire Line
+	10450 4000 10775 4000
+Wire Wire Line
+	10775 4000 10775 4100
+Connection ~ 4275 4525
+Wire Wire Line
+	4275 5075 4275 4975
+Wire Wire Line
+	4275 4525 4275 4675
+Wire Wire Line
+	4150 3800 4150 3925
+Connection ~ 4150 3925
+Wire Wire Line
+	4400 3800 4400 4025
+Connection ~ 4400 4025
+Wire Wire Line
+	4150 2700 4150 3500
+Connection ~ 5200 2700
+Wire Wire Line
+	4400 3500 4400 2700
+Connection ~ 4400 2700
+Text Notes 3400 3725 0    50   ~ 0
+OPTIONAL Weak\nPull-Up Resistors
 $EndSCHEMATC

Commit message: V2 is ready
Parts:
- added R4: 330k, Resistors_THT:R_Axial_DIN0207_L6.3mm_D2.5mm_P10.16mm_Horizontal, symbol R
- J1: value AMIGA_SIGNALS -> INPUT_SIGNALS
- renumbered R2 to R1, R3 to R2, R1 to R3
Connections:
- net GND: now also R4.2
- net at C1.1, R3.2, U1.11 (Cp)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: now also R4.1
Other:
- note added: "IN1"
- note added: "IN2"
- note added: "OUT1"
- note added: "OUT2"
- note removed: "LMB (Odd CIA Pin 8)"
- note removed: "RMB (Paula Pin 33)"
- moved on the sheet: C1, R3
Changed lines of the file:
@@
 Sheet 1 1
 Title "OpenAmigaMouseTrigger"
-Date "2018-01-07"
-Rev "1"
+Date "2018-05-29"
+Rev "2"
 Comp "SukkoPera"
 Comment1 ""
@@
 P 3750 3925
 F 0 "J1" H 3750 4025 50  0000 C CNN
-F 1 "AMIGA_SIGNALS" H 3800 3725 50  0000 C CNN
+F 1 "INPUT_SIGNALS" H 3750 3725 50  0000 C CNN
 F 2 "OpenAmigaMouseTrigger:LoosePads-2" H 3750 3925 50  0001 C CNN
 F 3 "" H 3750 3925 50  0001 C CNN
@@
 	-1   0    0    -1
 $EndComp
-Text Notes 2875 3950 0    50   ~ 0
-LMB (Odd CIA Pin 8)
-Text Notes 2900 4050 0    50   ~ 0
-RMB (Paula Pin 33)
+Text Notes 3550 3975 0    50   ~ 0
+IN1
+Text Notes 3550 4075 0    50   ~ 0
+IN2
 $Comp
 L C C1
 U 1 1 5A38359F
-P 4275 4825
-F 0 "C1" H 4300 4925 50  0000 L CNN
-F 1 "10u" H 4300 4725 50  0000 L CNN
-F 2 "Capacitors_THT:CP_Radial_D5.0mm_P2.00mm" H 4313 4675 50  0001 C CNN
-F 3 "" H 4275 4825 50  0001 C CNN
-	1    4275 4825
-	1    0    0    -1
-$EndComp
-$Comp
-L R R1
+P 3975 4825
+F 0 "C1" H 4000 4925 50  0000 L CNN
+F 1 "10u" H 4000 4725 50  0000 L CNN
+F 2 "Capacitors_THT:CP_Radial_D5.0mm_P2.00mm" H 4013 4675 50  0001 C CNN
+F 3 "" H 3975 4825 50  0001 C CNN
+	1    3975 4825
+	1    0    0    -1
+$EndComp
+$Comp
+L R R3
 U 1 1 5A3835EC
-P 3850 4525
-F 0 "R1" V 3930 4525 50  0000 C CNN
-F 1 "4.7k" V 3850 4525 50  0000 C CNN
-F 2 "Resistors_THT:R_Axial_DIN0207_L6.3mm_D2.5mm_P10.16mm_Horizontal" V 3780 4525 50  0001 C CNN
-F 3 "" H 3850 4525 50  0001 C CNN
-	1    3850 4525
+P 3550 4525
+F 0 "R3" V 3630 4525 50  0000 C CNN
+F 1 "4.7k" V 3550 4525 50  0000 C CNN
+F 2 "Resistors_THT:R_Axial_DIN0207_L6.3mm_D2.5mm_P10.16mm_Horizontal" V 3480 4525 50  0001 C CNN
+F 3 "" H 3550 4525 50  0001 C CNN
+	1    3550 4525
 	0    -1   -1   0
 $EndComp
@@
 L VCC #PWR01
 U 1 1 5A383C7B
-P 3475 4400
-F 0 "#PWR01" H 3475 4250 50  0001 C CNN
-F 1 "VCC" H 3475 4550 50  0000 C CNN
-F 2 "" H 3475 4400 50  0001 C CNN
-F 3 "" H 3475 4400 50  0001 C CNN
-	1    3475 4400
+P 3175 4400
+F 0 "#PWR01" H 3175 4250 50  0001 C CNN
+F 1 "VCC" H 3175 4550 50  0000 C CNN
+F 2 "" H 3175 4400 50  0001 C CNN
+F 3 "" H 3175 4400 50  0001 C CNN
+	1    3175 4400
 	1    0    0    -1
 $EndComp
@@
 P 7500 3925
 F 0 "J2" H 7500 4025 50  0000 C CNN
-F 1 "OUTPUT" H 7700 3875 50  0000 C CNN
+F 1 "OUTPUT" H 7500 3700 50  0000 C CNN
 F 2 "OpenAmigaMouseTrigger:LoosePads-2" H 7500 3925 50  0001 C CNN
 F 3 "" H 7500 3925 50  0001 C CNN
@@
 	1    0    0    -1
 $EndComp
-Text Notes 3500 4825 0    60   ~ 0
+Text Notes 3200 4825 0    60   ~ 0
 CLOCK PULSE\nGENERATOR
 $Comp
 L GND #PWR011
 U 1 1 5A385557
-P 4275 5075
-F 0 "#PWR011" H 4275 4825 50  0001 C CNN
-F 1 "GND" H 4275 4925 50  0000 C CNN
-F 2 "" H 4275 5075 50  0001 C CNN
-F 3 "" H 4275 5075 50  0001 C CNN
-	1    4275 5075
+P 4150 5125
+F 0 "#PWR011" H 4150 4875 50  0001 C CNN
+F 1 "GND" H 4150 4975 50  0000 C CNN
+F 2 "" H 4150 5125 50  0001 C CNN
+F 3 "" H 4150 5125 50  0001 C CNN
+	1    4150 5125
 	1    0    0    -1
 $EndComp
@@
 NoConn ~ 10950 6075
 $Comp
-L R R2
+L R R1
 U 1 1 5A528FE1
 P 4150 3650
-F 0 "R2" V 4230 3650 50  0000 C CNN
+F 0 "R1" V 4230 3650 50  0000 C CNN
 F 1 "22k" V 4150 3650 50  0000 C CNN
 F 2 "Resistors_THT:R_Axial_DIN0207_L6.3mm_D2.5mm_P10.16mm_Horizontal" V 4080 3650 50  0001 C CNN
@@
 $EndComp
 $Comp
-L R R3
+L R R2
 U 1 1 5A5291EB
 P 4400 3650
-F 0 "R3" V 4480 3650 50  0000 C CNN
+F 0 "R2" V 4480 3650 50  0000 C CNN
 F 1 "22k" V 4400 3650 50  0000 C CNN
 F 2 "Resistors_THT:R_Axial_DIN0207_L6.3mm_D2.5mm_P10.16mm_Horizontal" V 4330 3650 50  0001 C CNN
@@
 $EndComp
 Wire Wire Line
-	3475 4400 3475 4525
-Wire Wire Line
-	3475 4525 3700 4525
-Wire Wire Line
-	4000 4525 4875 4525
+	3175 4400 3175 4525
+Wire Wire Line
+	3175 4525 3400 4525
+Wire Wire Line
+	3700 4525 4875 4525
 Wire Wire Line
 	4875 3425 4875 4800
@@
 	3950 4025 4750 4025
 Wire Wire Line
-	6600 3225 7025 3225
-Wire Wire Line
-	7025 3225 7025 3925
-Wire Wire Line
-	7025 3925 7300 3925
+	6600 3225 7000 3225
+Wire Wire Line
+	7000 3225 7000 3925
+Wire Wire Line
+	7000 3925 7300 3925
 Wire Wire Line
 	7300 4025 7000 4025
@@
 Wire Wire Line
 	10775 4000 10775 4100
-Connection ~ 4275 4525
-Wire Wire Line
-	4275 5075 4275 4975
-Wire Wire Line
-	4275 4525 4275 4675
+Connection ~ 3975 4525
+Wire Wire Line
+	3975 4525 3975 4675
 Wire Wire Line
 	4150 3800 4150 3925
@@
 Text Notes 3400 3725 0    50   ~ 0
 OPTIONAL Weak\nPull-Up Resistors
+$Comp
+L R R4
+U 1 1 5ACFD32F
+P 4325 4825
+F 0 "R4" V 4405 4825 50  0000 C CNN
+F 1 "330k" V 4325 4825 50  0000 C CNN
+F 2 "Resistors_THT:R_Axial_DIN0207_L6.3mm_D2.5mm_P10.16mm_Horizontal" V 4255 4825 50  0001 C CNN
+F 3 "" H 4325 4825 50  0001 C CNN
+	1    4325 4825
+	1    0    0    -1
+$EndComp
+Wire Wire Line
+	4325 4675 4325 4525
+Connection ~ 4325 4525
+Wire Wire Line
+	3975 4975 3975 5075
+Wire Wire Line
+	3975 5075 4325 5075
+Wire Wire Line
+	4325 5075 4325 4975
+Wire Wire Line
+	4150 5125 4150 5075
+Connection ~ 4150 5075
+Text Notes 7575 3975 0    60   ~ 0
+OUT1
+Text Notes 7575 4075 0    60   ~ 0
+OUT2
 $EndSCHEMATC
